File: Through-Hole-Card.kicad_sch (KiCad schematic)
At the start: 8 parts, among them J1 Conn_01x02_Pin

Commit message: a
Other:
- note added: "Pin 5 i pin 4 e taşı Pin 5 de arıza veriyor yeni versionda bunu düzelt"
- note removed: "5V VIN Oluyor mu bak"
- note removed: "DS1302 mi ne o gelcek bir de 3 wire kullanıyor ona da bak"
- note removed: "Pinleri öncesinde bağla breadboardda sıkıntı veriyor mu bak"
Changed lines of the file:
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@@
     (stroke (width 0) (type default))
   )
-  (text "DS1302 mi ne o gelcek bir de 3 wire kullanıyor ona da bak\n"
-    (at 101.6 35.56 0)
+  (text "Pin 5 i pin 4 e taşı\nPin 5 de arıza veriyor yeni versionda bunu düzelt\n"
+    (at 100.33 38.1 0)
     (effects (font (size 1.27 1.27)) (justify left bottom))
   )
-  (text "Pinleri öncesinde bağla breadboardda sıkıntı veriyor mu bak\n"
-    (at 100.33 41.91 0)
-    (effects (font (size 1.27 1.27)) (justify left bottom))
-  )
-  (text "5V VIN Oluyor mu bak\n\n" (at 99.06 48.26 0)
-    (effects (font (size 1.27 1.27)) (justify left bottom))
-  )
