File: Through-Hole-Card.kicad_pcb (KiCad board)
At the start: 2 copper layers, 61 x 60 mm, 8 parts, among them J1 Conn_01x02_Pin

Commit message: a
Other:
- board text added: "ESP32 Wroom32"
- board text added: "RTC DS1302 Timer"
- board text added: "SD-Card Module"
Changed lines of the file:
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@@
     (property "Sheetname" "")
     (attr through_hole)
-    (fp_text reference "BME280_1" (at -1.8 -6.95 unlocked) (layer "F.SilkS")
+    (fp_text reference "BME280_1" (at 7.2344 -6.23 90 unlocked) (layer "F.SilkS")
         (effects (font (size 1 1) (thickness 0.1)))
     )
@@
     (property "Sheetname" "")
     (attr through_hole)
-    (fp_text reference "RTC_DS1302_1" (at 5 7 90 unlocked) (layer "B.SilkS")
+    (fp_text reference "RTC_DS1302_1" (at 8.0404 -21.9276 -180 unlocked) (layer "B.SilkS") hide
         (effects (font (size 1 1) (thickness 0.1)) (justify mirror))
     )
@@
   (gr_rect (start 131 51) (end 192 111)
     (stroke (width 0.1) (type default)) (fill none) (layer "Edge.Cuts"))
+  (gr_text "RTC DS1302 Timer " (at 164.0332 103.1748 180) (layer "B.SilkS")
+    (effects (font (size 1 1) (thickness 0.15)) (justify left bottom mirror))
+  )
+  (gr_text "SD-Card Module\n" (at 170.0276 67.31 90) (layer "B.SilkS")
+    (effects (font (size 1 1) (thickness 0.15)) (justify left bottom mirror))
+  )
+  (gr_text "ESP32 Wroom32 \n" (at 169.2656 86.4616 90) (layer "F.SilkS")
+    (effects (font (size 1 1) (thickness 0.15)) (justify left bottom))
+  )
   (segment (start 154.315 105.685) (end 164.5 95.5) (width 1) (layer "F.Cu") (net 1))
   (segment (start 156.93 63.43) (end 153.91 63.43) (width 1) (layer "F.Cu") (net 1))
@@
   (segment (start 144.595 87.905) (end 151.29 81.21) (width 0.25) (layer "B.Cu") (net 12))
   (segment (start 151.29 81.21) (end 153.91 81.21) (width 0.25) (layer "B.Cu") (net 12))
+  (segment (start 190.1 93.35) (end 190.1 68.6) (width 1) (layer "F.Cu") (net 13))
   (segment (start 190.1 68.6) (end 184.94 63.44) (width 1) (layer "B.Cu") (net 13))
   (segment (start 135 60.5) (end 164 60.5) (width 1) (layer "B.Cu") (net 13))
   (segment (start 179.832 59.944) (end 183.388 59.944) (width 1) (layer "B.Cu") (net 13))
-  (segment (start 190.1 93.35) (end 190.1 68.6) (width 1) (layer "B.Cu") (net 13))
   (segment (start 179 60.776) (end 179.832 59.944) (width 1) (layer "B.Cu") (net 13))
   (segment (start 166.94 63.44) (end 179 63.44) (width 1) (layer "B.Cu") (net 13))

Commit message: a
Parts:
- moved U3 0.09 mm to (151.5, 53.5)
- moved MPU6050_1 0.09 mm to (133.8, 107.0)
- moved SD_CARD1 0.06 mm to (132.1, 60.6)
